File: cc1125Carrier.kicad_sch (KiCad schematic)
At the start: 5 parts, among them J2 TFM-110-02-SM-D-A-K-TR, J3 Jumper Block, U1 YAAJ_WeAct_BlackPill_Part_Lik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

Commit message: update pullups on i2c, update images
Parts:
- added R1, R2: (no value), symbol Device:R
- J1: value (none) -> TFM-110-02-SM-D-A-K-TR; footprint (none) -> SamacSys_Parts:TFM-110-02-XXX-D-A-Y-TR
- J4: value (none) -> Conn_01x06; footprint (none) -> Connector_PinHeader_2.54mm:PinHeader_1x06_P2.54mm_Vertical
Connections:
- net MCU_VCC: now also R1.2, R2.2
- net SCL: now also R1.1
- net SDA: now also R2.1
